Commit message: updated some parameters

File: daxian_V2/urdf/daxian__hand_left_v1.urdf (robot description, URDF)
Before this commit: robot Left_hand_URDF_model, 23 links, 22 joints
Joints:
- joint left_hand_pinky_rota_joint: axis 0 0 -1 -> (none); limit lower=0 upper=1.57 effort=0.344 velocity=6.28 -> (none); type revolute -> fixed

File: daxian_V2/urdf/daxian__hand_right_v1.urdf (robot description, URDF)
Before this commit: robot Right_hand_URDF_model, 23 links, 22 joints
Joints:
- joint right_hand_pinky_rota_joint: axis 0 0 1 -> (none); limit lower=0 upper=1.57 effort=0.344 velocity=6.28 -> (none); type revolute -> fixed
